File: PCB/light-relay-module.kicad_pcb (KiCad board)
At the start: 2 copper layers, 142.8 x 86.9 mm, 164 parts, among them J1 Inputs, J2 DC, J3 Output, J4 Relays, J5 ICSP+, J6 ICSP+, J7 Relays, K1 FINDER-34.51, K10 FINDER-34.51, K2 FINDER-34.51, K3 FINDER-34.51, K4 FINDER-34.51, K5 FINDER-34.51, K6 FINDER-34.51, K7 FINDER-34.51, K8 FINDER-34.51, K9 FINDER-34.51, Q1 BTA16-800BW, Q10 BTA16-800BW, Q11 IRF7241, Q2 BTA16-800BW, Q3 BTA16-800BW, Q4 BTA16-800BW, Q5 BTA16-800BW, Q6 BTA16-800BW, Q7 BTA16-800BW, Q8 BTA16-800BW, Q9 BTA16-800BW, SW1 TRIAC TEST, U1 TLP627-2, U10 VOT8024AG, U11 VOT8024AG, U12 VOT8024AG, U13 74LVC1G125, U14 VOT8024AG, U15 VOT8024AG, U16 VOT8024AG, U17 VOT8024AG, U18 VOT8024AG, U19 74HC595, U2 TLP627-2, U20 74HC595, U21 74HC595, U22 ULN2003A, U23 ULN2003A, U3 TLP627-2, U4 TLP627-2, U5 TLP627-2, U6 R-78E5.0-0.5, U7 ATmega644PA-M, U8 VOT8024AG, U9 VOT8024AG, Y1 8Mhz

Commit message: Add BOM, rename optocouplers
Parts:
- U1, U2, U3, U4, U5: value TLP627-2 -> MOCD223M
Changed lines of the file:
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@@
       (effects (font (size 0.7 0.7) (thickness 0.1)))
     )
-    (fp_text value "TLP627-2" (at -13.4566 -17.5758 180) (layer "F.Fab")
+    (fp_text value "MOCD223M" (at -13.4566 -17.5758 180) (layer "F.Fab")
       (effects (font (size 1 1) (thickness 0.15)))
     )
@@
       (effects (font (size 0.7 0.7) (thickness 0.1)))
     )
-    (fp_text value "TLP627-2" (at -15.0314 -23.2146 180) (layer "F.Fab")
+    (fp_text value "MOCD223M" (at -15.0314 -23.2146 180) (layer "F.Fab")
       (effects (font (size 1 1) (thickness 0.15)))
     )
@@
       (effects (font (size 0.7 0.7) (thickness 0.1)))
     )
-    (fp_text value "TLP627-2" (at -16.6062 -28.9042 180) (layer "F.Fab")
+    (fp_text value "MOCD223M" (at -16.6062 -28.9042 180) (layer "F.Fab")
       (effects (font (size 1 1) (thickness 0.15)))
     )
@@
       (effects (font (size 0.7 0.7) (thickness 0.1)))
     )
-    (fp_text value "TLP627-2" (at -20.0098 -40.0294 180) (layer "F.Fab")
+    (fp_text value "MOCD223M" (at -20.0098 -40.0294 180) (layer "F.Fab")
       (effects (font (size 1 1) (thickness 0.15)))
     )
@@
       (effects (font (size 0.7 0.7) (thickness 0.1)))
     )
-    (fp_text value "TLP627-2" (at -18.181 -34.4414 180) (layer "F.Fab")
-      (effects (font (size 1 1) (thickness 0.15)))
-    )
+    (fp_text value "MOCD223M" (at -18.181 -34.4414 180) (layer "F.Fab")
+      (effects (font (size 1 1) (thickness 0.15)))
+    )
