File: PCB/light-relay-module.kicad_sch (KiCad schematic)
At the start: 164 parts, among them J1 Inputs, J2 DC, J3 Output, J4 Relays, J5 ICSP+, J6 ICSP+, J7 Relays, K1 FINDER-34.51, K10 FINDER-34.51, K2 FINDER-34.51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

Commit message: Add BOM, rename optocouplers
Parts:
- U1, U2, U3, U4, U5: value TLP627-2 -> MOCD223M
Other:
- note added: "OE buffer"
- note added: "Test button"
- moved on the sheet: C5, C6, R22, R28, R29, R76, SW1, U13
